File: dcdc.sch (KiCad schematic (older format))
At the start: 40 parts, among them J1 SOLAR, J2 LOAD, J3 BAT, Q1 PSMN5R2-60YLX, Q2 PSMN5R2-60YLX, Q3 PSMN5R2-60YLX, Q4 PSMN5R2-60YLX, T1 MMBT3904, U1 LM5109BMA

Commit message: Several improvements (v0.4) after first tests
- Ultra-low-power MCU STM32L072
- Larger screw terminals
- USB power supply replaced by more efficient SMPS
- High-side load switch with P-MOS
- High-side current measurement to include USB current in load measurement
Parts:
- removed C2: 680u, Capacitor_THT:CP_Radial_D16.0mm_P7.50mm, symbol Project:CP
- removed R12: 2.2k, LibreSolar:R_0603_1608, symbol Project:R
- added C11, C13, C17, C18: 10n, LibreSolar:C_0603_1608, symbol Project:C
- added C16, C42, C9: 100n, LibreSolar:C_0603_1608, symbol Project:C
- added J6: PWR_12V, Connector_PinHeader_2.54mm:PinHeader_1x02_P2.54mm_Vertical, symbol Connector:Conn_01x02_Male
- added R11, R20: 2.2k, LibreSolar:R_0603_1608, symbol Project:R
- added R23: 10k, LibreSolar:R_0603_1608, symbol Project:R
- added R24, R25: 100k, LibreSolar:R_0603_1608, symbol Project:R
- added R26, R27: 5.6k, LibreSolar:R_0603_1608, symbol Project:R
- added RT1: 10k, LibreSolar:R_0603_1608, symbol Device:Thermistor_NTC
- added TP1, TP2, TP3, TP4, TP5, TP6: Test_Point_Probe, TestPoint:TestPoint_Pad_D1.0mm, symbol Connector:TestPoint_Probe
- added U6: INA2181, LibreSolar:VSSOP-10_3.0x3.0mm_P0.5mm, symbol Project:INA2181
- C1: value 680u -> 1200u; footprint Capacitor_THT:CP_Radial_D16.0mm_P7.50mm -> LibreSolar:CP_Radial_L31.5mm_D16.0mm_P7.50mm_horizontal; Alternative Panasonic EEU-FR1J561SB -> (none); PartNumber EKYB630ELL681ML20S -> EKYB630ELL122MLN3S; Remarks 63V, 2.25A, 16x20 -> 63V, 3.0A, 16x31.5
- D3, D6: Config (none) -> +testing; DNP (none) -> X
- J1, J2, J3: footprint LibreSolar:Phoenix_Contact_PT_2,5-2-7,5-H -> LibreSolar:Phoenix_Contact_MKDS_5-2-7,62; PartNumber 1988105 -> 1868076
- L1: footprint LibreSolar:L-FERYSTER-DTMSS-27 -> LibreSolar:L-FERYSTER-DTMSS-27_33uH
- Q3: value PSMN5R2-60YLX -> BSC084P03NS3; symbol Project:Q_NMOS -> LibreSolar:Q_PMOS; Alternative (none) -> SI7149ADP-T1-GE3; Manufacturer Nexperia -> Infineon; PartNumber PSMN5R2-60YLX -> BSC084P03NS3GATMA1
- R9: value 56k -> 10k; PartNumber RC0603FR-0756KL -> RC0603FR-0710KL
Connections:
- net +12V: now also R17.1, R6.2, R25.1, TP1.1, U6.2 (IN-1), U6.7 (IN+2); no longer C12.1, C27.1, C37.1, C5.1, D5.1 (K), J2.2, L1.2, R10.2, R9.2, U1.1 (VDD)
- net DCDC_IN: now also R24.1
- net GND: now also C27.2, C7.2, D5.2 (A), J2.2, J3.2, R4.1, T1.2 (E), C11.2, C13.2, C16.2, C17.2, C18.2, C42.2, C9.2, J6.2 (Pin_2), R26.2, R27.2, RT1.2, U6.4 (GND); no longer C6.2, R6.1
- net PWM_HS: now also TP2.1
- net PWM_LS: now also TP3.1
- net SW_NODE: now also C6.1; no longer R4.2
- net at T1.3 (C): now also R16.1; no longer R9.1
- net at Q3.G: now also C28.2, R16.2, R9.1; no longer C28.1
- net at R13.1, T1.1 (B): no longer R16.2
- removed net BAT-: C7.2, J3.2, R17.1, R6.2
- removed net LOAD-: C27.2, C28.2, D5.2 (A), J2.1, Q3.D
- net LOAD-SW renamed LOAD_S
- net LOAD_S: now also R9.2, J6.1 (Pin_1), U6.8 (IN-2); no longer R16.1, T1.2 (E)
- net ~LOAD_EN renamed LOAD_EN
- new net: C6.2, R4.2
- new net: R11.1, U6.9 (OUT2)
- new net: R20.1, U6.1 (OUT1)
- new net +10V: C12.1, R10.2, U1.1 (VDD)
- new net +3V3: C9.1, R23.1, U6.10 (VS)
- new net DAC: C42.1, TP6.1, U6.5 (REF1), U6.6 (REF2)
- new net DCDC_OUT: C37.1, C5.1, L1.2, R6.1, U6.3 (IN+1)
- new net I_DCDC: C13.1, R20.2, TP4.1
- new net I_LOAD: C11.1, R11.2, TP5.1
- new net LOAD+: C27.1, C28.1, D5.1 (K), J2.1, Q3.D
- new net T_MOSFETS: C16.1, R23.2, RT1.1
- new net V_BAT: C18.1, R25.2, R27.1
- new net V_SOLAR: C17.1, R24.2, R26.1
- no-connect marks 1 -> 0
Other:
- note added: "Current sense amplifier"
- note added: "Diff. amp. reference\ndefined by DAC pin\ninstead of GND: variable\nzero current set point"
- note added: "High-side switch necessary, \notherwise e.g. in case of\na laptop powered by 12V and \nconnected to USB port\nGND current would continue \nthrough USB wire."
- note added: "MOSFET\ntemperature"
- note added: "Same voltage divider to use COMP1 for\nMCU wake-up when Vsolar > Vbat"
- note added: "Solar and battery voltage"
- note removed: "Alternative: 330R at MOSFET gate\n--> 10.4/330 = 31 mA max"
- note removed: "typisch: 1-10 nF + 10 uF"
- moved on the sheet: C1, C10, C12, C27, C28, C3, C37, C4, C5, C6, C7, C8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

Commit message: Board shape adjusted and 6P6C connector added
Parts:
- removed C16: 100n, LibreSolar:C_0603_1608, symbol Project:C
- removed R23: 10k, LibreSolar:R_0603_1608, symbol Project:R
- removed RT1: 10k, LibreSolar:R_0603_1608, symbol Device:Thermistor_NTC
- D3, D6: Alternative Nexperia PMEG4010EGWX -> (none); Config +testing -> (none); DNP X -> (none); Remarks (none) -> Alternative: Nexperia PMEG4010EGWX
- F1: footprint LibreSolar:Fuse_Clip_5x20mm -> LibreSolar:KEYSTONE-FUSE-3557-2; Alternative Littelfuse 01110501Z, Keystone 3521 -> (none); Manufacturer Bel fuse -> Keystone; PartNumber FC-203 bright tin -> 3557-2; Remarks Order 2x clip + fuse Littelfuse 0217015.MXP -> (none)
- J1: value SOLAR -> MKDS_5-2_952; footprint LibreSolar:Phoenix_Contact_MKDS_5-2-7,62 -> LibreSolar:Phoenix_Contact_MKDS_5-2-952; PartNumber 1868076 -> 1714971
- J2: value LOAD -> MKDS_5-2_952; footprint LibreSolar:Phoenix_Contact_MKDS_5-2-7,62 -> LibreSolar:Phoenix_Contact_MKDS_5-2-952; PartNumber 1868076 -> 1714971
- J3: value BAT -> MKDS_5-2_952; footprint LibreSolar:Phoenix_Contact_MKDS_5-2-7,62 -> LibreSolar:Phoenix_Contact_MKDS_5-2-952; PartNumber 1868076 -> 1714971
- J6: footprint Connector_PinHeader_2.54mm:PinHeader_1x02_P2.54mm_Vertical -> Connector_JST:JST_XH_B02B-XH-A_1x02_P2.50mm_Vertical; symbol Connector:Conn_01x02_Male -> Connector_Generic:Conn_01x02; Manufacturer (none) -> JST; PartNumber (none) -> B2B-XH-A (LF)(SN)
- Q1, Q2, Q4: Remarks (none) -> Alternative: BUK9Y6R0-60E
- Q3: Alternative SI7149ADP-T1-GE3 -> (none); Remarks (none) -> Alternative: SI7149ADP-T1-GE3
- R17, R6: value 4m -> 3m; PartNumber CRE2512-FZ-R004E-3 -> CRE2512-FZ-R003E-3
- U1: symbol Project:LM5109B -> Project:LM5109BMA
Connections:
- net DCDC_OUT: now also R10.2
- net at D4.2 (A), R10.1: now also C12.1, U1.1 (VDD)
- removed net +10V: C12.1, R10.2, U1.1 (VDD)
- net DCDC_IN renamed SOLAR+
Other:
- note removed: "MOSFET\ntemperature"
- moved on the sheet: D4, R10

Commit message: Solar voltage input protection added
Parts:
- added Q7: BSS83P, LibreSolar:SOT-23, symbol Device:Q_PMOS_GSD
- added R31, R36: 10k, LibreSolar:R_0603_1608, symbol Project:R
- added R32: 1M, LibreSolar:R_0603_1608, symbol Project:R
- added T2: MMBT3904, LibreSolar:SOT-23, symbol Transistor_BJT:BC817
Connections:
- net GND: now also T2.2 (E)
- net SOLAR+: now also Q7.2 (S), R32.1; no longer R24.1
- new net: Q7.3 (D), R24.1
- new net: Q7.1 (G), R32.2, R36.2
- new net: R31.1, T2.1 (B)
- new net: R36.1, T2.3 (C)
- new net V_SOLAR_EN: R31.2
Other:
- note added: "Battery voltage"
- note added: "PMOS for protection\nof MCU pins if PV\npanel is connected\nbefore battery"
- note added: "Same voltage divider for V_SOLAR\nand V_BAT to use COMP1 for MCU\nwake-up when Vsolar > Vbat"
- note added: "Solar voltage"
- note removed: "Same voltage divider to use COMP1 for\nMCU wake-up when Vsolar > Vbat"
- note removed: "Solar and battery voltage"
- moved on the sheet: C10, C12, C17, C18, D4, J6, R10, R24, R25, R26, R27, TP2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
