File: kicad/mcu.sch (KiCad schematic (older format))
At the start: 35 parts, among them J4 UEXT, J7 6P6C, J8 ST_Nucleo_SWD, U2 STM32L072CZT6, U3 D1213A-04SO

Commit message: Small changes and files renamed
Connections:
- net +3V3: no longer R35.1
- net BOOT0: now also C43.1, R33.2, R35.2, R7.2; no longer R7.1
- net BUTTON: now also R7.1; no longer C43.1, R33.2, R35.2
- net GND: now also R35.1; no longer R7.2
Other:
- note added: "BUTTON can trigger bootloader\nif pulled high before reset.\nDuration of high input on BOOT0:\n\ntau = R35 * C43\nV(t) = Vmax * (1-exp(-t/tau))\n--> t = -tau * ln(1-V/Vmax)\n\nV > 0.7 * VDD = 2.31V necessary\n--> t = 12 ms"
- note added: "LED1 could becontrolled\nby LPTIM1_OUT in stop\nmode --> use PB2"
- note added: "Pull-up to provide defined RX\nsignal if port is unconnected"
- note removed: "LED1 controlled by LPTIM1_OUT\nin stop mode: only PB2 possible"
- moved on the sheet: C24, C43, C44, F2, J7, R18, R19, R21, R22, R33, R34, R35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

Commit message: Small adjustments after testing
- MOSFET gate driver changed to reduce switch node ringing
- Current measurement output filter time constant reduced to have less delay
- BTN pin allows starting the bootloader if pulled to 3V3 before startup
Parts:
- C44: Manufacturer Yageo -> Murata
Other:
- note added: "Either internal SMD NTC on PCB or\nexternal sensor via 6P6C connector"
- note added: "LED1 could be controlled\nby LPTIM1_OUT in stop\nmode --> use PB2"
- note added: "LS.one interface"
- note added: "Temperature\n(ext. or int.)"
- note removed: "Either internal SMD NTC\nsoldered or external \nsensor via 6P6C connector"
- note removed: "LED1 could becontrolled\nby LPTIM1_OUT in stop\nmode --> use PB2"
- note removed: "Serial interface"
- note removed: "Temperature\n(external or \ninternal)"
Changed lines of the file:
@@
 encoding utf-8
 Sheet 3 4
-Title "10A MPPT Charge Controller with USB"
-Date "2019-06-03"
-Rev "0.6.1"
-Comp "Libre Solar / Connected Energy"
+Title "MPPT 1210 HUS"
+Date "2019-07-24"
+Rev "0.7.1"
+Comp "Libre Solar"
 Comment1 "Author: Martin Jäger"
 Comment2 "Website: https://libre.solar"
@@
 Text Notes 2800 1250 0    100  ~ 0
 MCU STM32L072
-Text Notes 9700 1000 0    100  ~ 0
+Text Notes 9400 1000 0    100  ~ 0
 STM Nucleo SWD
 Text Label 1600 4300 0    50   ~ 0
@@
 L power:+3.3V #PWR0101
 U 1 1 5AE4F2FA
-P 5700 1400
-F 0 "#PWR0101" H 5700 1250 50  0001 C CNN
-F 1 "+3.3V" H 5700 1540 50  0000 C CNN
-F 2 "" H 5700 1400 50  0000 C CNN
-F 3 "" H 5700 1400 50  0000 C CNN
-	1    5700 1400
+P 5700 1500
+F 0 "#PWR0101" H 5700 1350 50  0001 C CNN
+F 1 "+3.3V" H 5700 1640 50  0000 C CNN
+F 2 "" H 5700 1500 50  0000 C CNN
+F 3 "" H 5700 1500 50  0000 C CNN
+	1    5700 1500
 	1    0    0    -1
 $EndComp
@@
 	1    0    0    -1
 $EndComp
-Text Notes 6100 1000 0    100  ~ 0
+Text Notes 5800 1000 0    100  ~ 0
 UEXT connector
 Text Notes 7850 1000 0    100  ~ 0
@@
 	5700 1600 5900 1600
 Wire Wire Line
-	5700 1600 5700 1400
+	5700 1600 5700 1500
 Text Label 4000 4100 2    50   ~ 0
 I2C1_SDA
@@
 	2200 3500 1600 3500
 Text Notes 4150 3850 0    50   ~ 0
-LED1 could becontrolled\nby LPTIM1_OUT in stop\nmode --> use PB2
+LED1 could be controlled\nby LPTIM1_OUT in stop\nmode --> use PB2
 Wire Wire Line
 	2200 3900 1600 3900
@@
 	0    1    1    0
 $EndComp
-$Comp
-L power:GND #PWR04
-U 1 1 5BA050D5
-P 4800 2700
-F 0 "#PWR04" H 4800 2450 50  0001 C CNN
-F 1 "GND" H 4800 2550 50  0000 C CNN
-F 2 "" H 4800 2700 50  0000 C CNN
-F 3 "" H 4800 2700 50  0000 C CNN
-	1    4800 2700
-	1    0    0    -1
-$EndComp
-Text Label 4800 2100 3    50   ~ 0
-BOOT0
-Wire Wire Line
-	4800 2400 4800 2100
-Wire Wire Line
-	4800 2600 4800 2700
 Text Notes 1250 1550 0    50   ~ 0
 Measured current into\nVDDA around 1.2 mA
@@
 F 2 "LibreSolar:C_0603_1608" H 8800 5700 50  0001 C CNN
 F 3 "" H 8825 5975 50  0000 C CNN
-F 4 "Yageo" H 0   50  50  0001 C CNN "Manufacturer"
+F 4 "Murata" H 0   50  50  0001 C CNN "Manufacturer"
 F 5 "GCM188R72A103KA37D" H -500 100 50  0001 C CNN "PartNumber"
 	1    8800 5900
@@
 Connection ~ 8000 5600
 Text Notes 9300 5650 0    100  ~ 0
-Temperature\n(external or \ninternal)
+Temperature\n(ext. or int.)
 Text GLabel 8900 5600 2    50   Output ~ 0
 T_BAT
@@
 Text Label 7350 5600 0    50   ~ 0
 TEMP_EXT
-Text Notes 9150 6100 0    50   ~ 0
-Either internal SMD NTC\nsoldered or external \nsensor via 6P6C connector
+Text Notes 9300 6100 0    50   ~ 0
+Either internal SMD NTC on PCB or\nexternal sensor via 6P6C connector
 Text Notes 7100 2600 0    100  ~ 0
-Serial interface
+LS.one interface
 Wire Wire Line
 	7300 3900 7300 4000
